Commit message: Rebase from 'upstream'

File: rm_description/urdf/balance/balance.urdf.xacro (robot description, xacro)
@@ -1,43 +1,24 @@
 <?xml version="1.0"?>
 <robot xmlns:xacro="http://www.ros.org/wiki/xacro" name="balance">
-  <xacro:arg name="load_chassis" default="true"/>
-  <xacro:arg name="load_gimbal" default="true"/>
-  <xacro:arg name="load_shooter" default="true"/>
-  <xacro:arg name="use_simulation" default="true"/>
-  <xacro:if value="$(arg load_chassis)">
-    <xacro:include filename="$(find rm_description)/urdf/balance/chassis.urdf.xacro"/>
-    <xacro:chassis/>
-  </xacro:if>
-  <xacro:if value="$(arg load_gimbal)">
-  </xacro:if>
-  <xacro:if value="$(arg load_shooter)">
-  </xacro:if>
-  <xacro:if value="$(arg use_simulation)">
-    <gazebo>
-      <plugin name="rm_ros_control" filename="librm_robot_hw_sim.so">
-        <robotNamespace>/</robotNamespace>
-        <robotSimType>rm_gazebo/RmRobotHWSim</robotSimType>
-      </plugin>
-    </gazebo>
-    <gazebo reference="base_link">
-      <gravity>true</gravity>
-      <sensor name="imu_sensor" type="imu">
-        <always_on>true</always_on>
-        <update_rate>1000</update_rate>
-        <visualize>true</visualize>
-        <topic>__default_topic__</topic>
-        <plugin filename="libgazebo_ros_imu_sensor.so" name="imu_plugin">
-          <topicName>base_imu</topicName>
-          <bodyName>imu_link</bodyName>
-          <updateRateHZ>1000.0</updateRateHZ>
-          <gaussianNoise>0.0</gaussianNoise>
-          <xyzOffset>0 0 0</xyzOffset>
-          <rpyOffset>0 0 0</rpyOffset>
-          <frameName>imu_link</frameName>
-          <initialOrientationAsReference>false</initialOrientationAsReference>
-        </plugin>
-        <pose>0 0 0 0 0 0</pose>
-      </sensor>
-    </gazebo>
-  </xacro:if>
+    <xacro:arg name="load_chassis" default="true"/>
+    <xacro:arg name="load_gimbal" default="true"/>
+    <xacro:arg name="load_shooter" default="true"/>
+    <xacro:arg name="use_simulation" default="true"/>
+    <xacro:if value="$(arg load_chassis)">
+        <xacro:include filename="$(find rm_description)/urdf/balance/chassis.urdf.xacro"/>
+        <xacro:chassis/>
+        <xacro:IMU connected_to="base_link" imu_name="base_imu" xyz="0.08 0. 0.08" rpy="0 0 0"/>
+        <xacro:if value="$(arg load_gimbal)">
+            <xacro:if value="$(arg load_shooter)">
+            </xacro:if>
+        </xacro:if>
+    </xacro:if>
+    <xacro:if value="$(arg use_simulation)">
+        <gazebo>
+            <plugin name="rm_ros_control" filename="librm_robot_hw_sim.so">
+                <robotNamespace>/</robotNamespace>
+                <robotSimType>rm_gazebo/RmRobotHWSim</robotSimType>
+            </plugin>
+        </gazebo>
+    </xacro:if>
 </robot>

File: rm_description/urdf/common/imu.urdf.xacro (robot description, xacro)
@@ -1,21 +1,5 @@
 <?xml version="1.0"?>
-<!-- This file contains plugins to simulate an Imu sensor attached to the robot. -->
-<!-- Documentation can be found at http://wiki.ros.org/hector_gazebo_plugins -->
 <robot xmlns:xacro="http://www.ros.org/wiki/xacro" name="imu">
-    <xacro:macro name="IMU" params="connected_to imu_name simulation xyz:='0 0 0' rpy:='0 0 0' ">
-        <xacro:property name="imu_update_rate" value="200"/>
-        <xacro:property name="imu_calibration_service_name" value="${imu_name}/calibrate"/>
-        <xacro:property name="acceleration_offset" value="0.0 0.0 0.0"/>
-        <xacro:property name="acceleration_drift" value="0.0 0.0 0.0"/>
-        <xacro:property name="acceleration_drift_frequency" value="0.0 0.0 0.0"/>
-        <xacro:property name="acceleration_gaussian_noise" value="0.1 0.1 0.1"/>
-        <xacro:property name="rate_offset" value="0.0 0.0 0.0"/>
-        <xacro:property name="rate_drift" value="0.0 0.0 0.0"/>
-        <xacro:property name="rate_drift_frequency" value="0.0 0.0 0.0"/>
-        <xacro:property name="rate_gaussian_noise" value="0.2 0.2 0.2"/>
-        <xacro:property name="heading_offset" value="0.0"/>
-        <xacro:property name="heading_drift" value="0.0"/>
-        <xacro:property name="heading_drift_frequency" value="0.0"/>
-        <xacro:property name="heading_gaussian_noise" value="0.3"/>
+    <xacro:macro name="IMU" params="connected_to imu_name xyz:='0 0 0' rpy:='0 0 0' ">
         <!-- Imu is fixed to the base link -->
         <joint name="${imu_name}_joint" type="fixed">
@@ -47,27 +31,4 @@
             <disableFixedJointLumping>true</disableFixedJointLumping>
         </gazebo>
-        <xacro:if value="${simulation}">
-            <gazebo>
-                <plugin name="smb_imu_plugin" filename="libhector_gazebo_ros_imu.so">
-                    <updateRate>${imu_update_rate}</updateRate>
-                    <bodyName>${imu_name}</bodyName>
-                    <frameId>${imu_name}</frameId>
-                    <topicName>${imu_name}</topicName>
-                    <serviceName>${imu_calibration_service_name}</serviceName>
-                    <accelOffset>${acceleration_offset}</accelOffset>
-                    <accelDrift>${acceleration_drift}</accelDrift>
-                    <accelDriftFrequency>${acceleration_drift_frequency}</accelDriftFrequency>
-                    <accelGaussianNoise>${acceleration_gaussian_noise}</accelGaussianNoise>
-                    <rateOffset>${rate_offset}</rateOffset>
-                    <rateDrift>${rate_drift}</rateDrift>
-                    <rateDriftFrequency>${rate_drift_frequency}</rateDriftFrequency>
-                    <rateGaussianNoise>${rate_gaussian_noise}</rateGaussianNoise>
-                    <headingOffset>${heading_offset}</headingOffset>
-                    <headingDrift>${heading_drift}</headingDrift>
-                    <headingDriftFrequency>${heading_drift_frequency}</headingDriftFrequency>
-                    <headingGaussianNoise>${heading_gaussian_noise}</headingGaussianNoise>
-                </plugin>
-            </gazebo>
-        </xacro:if>
     </xacro:macro>
 </robot>

File: rm_description/urdf/hero/hero.urdf.xacro (robot description, xacro)
@@ -1,39 +1,38 @@
 <?xml version="1.0"?>
 <robot xmlns:xacro="http://www.ros.org/wiki/xacro" name="hero">
-  <xacro:arg name="load_chassis" default="true"/>
-  <xacro:arg name="load_gimbal" default="true"/>
-  <xacro:arg name="load_shooter" default="true"/>
-  <xacro:arg name="camera_link" default="camera_link"/>
-  <xacro:arg name="camera_optical_frame" default="camera_optical_frame"/>
-  <xacro:arg name="use_simulation" default="true"/>
-  <xacro:arg name="roller_type" default="realistic"/>
-  <xacro:if value="$(arg load_chassis)">
-    <xacro:include filename="$(find rm_description)/urdf/hero/chassis.urdf.xacro"/>
-    <xacro:chassis roller_type="$(arg roller_type)"/>
-  </xacro:if>
-  <xacro:if value="$(arg load_gimbal)">
-    <xacro:include filename="$(find rm_description)/urdf/hero/gimbal.urdf.xacro"/>
-    <xacro:include filename="$(find rm_description)/urdf/hero/gimbal.transmission.urdf.xacro"/>
-    <xacro:include filename="$(find rm_description)/urdf/common/imu.urdf.xacro"/>
-    <xacro:IMU connected_to="yaw" imu_name="gimbal_imu" simulation="true"
-               xyz="0.024 -0.014 0.088" rpy="0 ${pi/2} 0"/>
-    <xacro:include filename="$(find rm_description)/urdf/common/camera.urdf.xacro"/>
-    <xacro:camera_sensor xyz="0.05 0 -0.07" rpy="${pi} 0 -0.02" frame_id="$(arg camera_link)" parent="pitch"
-                         camera_sim="$(arg use_simulation)"/>
-    <xacro:camera_optical_frame xyz="0.2527 0.0071 -0.0984" rpy="1.5486 -0.0025 1.600"
-                                frame_id="$(arg camera_optical_frame)" parent="pitch"
-                                camera_sim="$(arg use_simulation)"/>
-  </xacro:if>
-  <xacro:if value="$(arg load_shooter)">
-    <xacro:include filename="$(find rm_description)/urdf/hero/shooter.urdf.xacro"/>
-    <xacro:include filename="$(find rm_description)/urdf/hero/shooter.transmission.urdf.xacro"/>
-  </xacro:if>
-  <xacro:if value="$(arg use_simulation)">
-    <gazebo>
-      <plugin name="rm_ros_control" filename="librm_robot_hw_sim.so">
-        <robotNamespace>/</robotNamespace>
-        <robotSimType>rm_gazebo/RmRobotHWSim</robotSimType>
-      </plugin>
-    </gazebo>
-  </xacro:if>
+    <xacro:arg name="load_chassis" default="true"/>
+    <xacro:arg name="load_gimbal" default="true"/>
+    <xacro:arg name="load_shooter" default="true"/>
+    <xacro:arg name="camera_link" default="camera_link"/>
+    <xacro:arg name="camera_optical_frame" default="camera_optical_frame"/>
+    <xacro:arg name="use_simulation" default="true"/>
+    <xacro:arg name="roller_type" default="realistic"/>
+    <xacro:if value="$(arg load_chassis)">
+        <xacro:include filename="$(find rm_description)/urdf/hero/chassis.urdf.xacro"/>
+        <xacro:chassis roller_type="$(arg roller_type)"/>
+        <xacro:if value="$(arg load_gimbal)">
+            <xacro:include filename="$(find rm_description)/urdf/hero/gimbal.urdf.xacro"/>
+            <xacro:include filename="$(find rm_description)/urdf/hero/gimbal.transmission.urdf.xacro"/>
+            <xacro:include filename="$(find rm_description)/urdf/common/imu.urdf.xacro"/>
+            <xacro:include filename="$(find rm_description)/urdf/common/camera.urdf.xacro"/>
+            <xacro:camera_sensor xyz="0.05 0 -0.07" rpy="${pi} 0 -0.02" frame_id="$(arg camera_link)" parent="pitch"
+                                 camera_sim="$(arg use_simulation)"/>
+            <xacro:camera_optical_frame xyz="0.2527 0.0071 -0.0984" rpy="1.5486 -0.0025 1.600"
+                                        frame_id="$(arg camera_optical_frame)" parent="pitch"
+                                        camera_sim="$(arg use_simulation)"/>
+            <xacro:IMU connected_to="pitch" imu_name="gimbal_imu" xyz="0.08 0. 0.08" rpy="0 0 -${pi/2}"/>
+            <xacro:if value="$(arg load_shooter)">
+                <xacro:include filename="$(find rm_description)/urdf/hero/shooter.urdf.xacro"/>
+                <xacro:include filename="$(find rm_description)/urdf/hero/shooter.transmission.urdf.xacro"/>
+            </xacro:if>
+        </xacro:if>
+    </xacro:if>
+    <xacro:if value="$(arg use_simulation)">
+        <gazebo>
+            <plugin name="rm_ros_control" filename="librm_robot_hw_sim.so">
+                <robotNamespace>/</robotNamespace>
+                <robotSimType>rm_gazebo/RmRobotHWSim</robotSimType>
+            </plugin>
+        </gazebo>
+    </xacro:if>
 </robot>

File: rm_description/urdf/standard3/standard3.urdf.xacro (robot description, xacro)
@@ -12,20 +12,19 @@
         <xacro:chassis roller_type="$(arg roller_type)"/>
         <xacro:include filename="$(find rm_description)/urdf/common/imu.urdf.xacro"/>
-        <xacro:IMU connected_to="base_link" imu_name="base_imu" simulation="true"
-                   xyz="0.0 -0.165 0.0" rpy="0 0 ${pi}"/>
-    </xacro:if>
-    <xacro:if value="$(arg load_gimbal)">
-        <xacro:include filename="$(find rm_description)/urdf/standard/gimbal.urdf.xacro"/>
-        <xacro:include filename="$(find rm_description)/urdf/standard3/gimbal.transmission.urdf.xacro"/>
-        <xacro:include filename="$(find rm_description)/urdf/common/camera.urdf.xacro"/>
-        <xacro:camera_sensor xyz="0.127 0 -0.038" rpy="0 0 0" frame_id="$(arg camera_link)" parent="pitch"
-                             camera_sim="$(arg use_simulation)"/>
-        <xacro:camera_optical_frame xyz="0.089 -0.004 -0.053" rpy="1.593 0.0 1.567"
-                                    frame_id="$(arg camera_optical_frame)" parent="pitch"
-                                    camera_sim="$(arg use_simulation)"/>
-    </xacro:if>
-    <xacro:if value="$(arg load_shooter)">
-        <xacro:include filename="$(find rm_description)/urdf/standard/shooter.urdf.xacro"/>
-        <xacro:include filename="$(find rm_description)/urdf/standard3/shooter.transmission.urdf.xacro"/>
+        <xacro:if value="$(arg load_gimbal)">
+            <xacro:include filename="$(find rm_description)/urdf/standard/gimbal.urdf.xacro"/>
+            <xacro:include filename="$(find rm_description)/urdf/standard3/gimbal.transmission.urdf.xacro"/>
+            <xacro:include filename="$(find rm_description)/urdf/common/camera.urdf.xacro"/>
+            <xacro:camera_sensor xyz="0.127 0 -0.038" rpy="0 0 0" frame_id="$(arg camera_link)" parent="pitch"
+                                 camera_sim="$(arg use_simulation)"/>
+            <xacro:camera_optical_frame xyz="0.089 -0.004 -0.053" rpy="1.593 0.0 1.567"
+                                        frame_id="$(arg camera_optical_frame)" parent="pitch"
+                                        camera_sim="$(arg use_simulation)"/>
+            <xacro:IMU connected_to="pitch" imu_name="gimbal_imu" xyz="0.08 0. 0.08" rpy="0 0 -${pi/2}"/>
+            <xacro:if value="$(arg load_shooter)">
+                <xacro:include filename="$(find rm_description)/urdf/standard/shooter.urdf.xacro"/>
+                <xacro:include filename="$(find rm_description)/urdf/standard3/shooter.transmission.urdf.xacro"/>
+            </xacro:if>
+        </xacro:if>
     </xacro:if>
     <xacro:if value="$(arg use_simulation)">

File: rm_description/urdf/standard4/standard4.urdf.xacro (robot description, xacro)
@@ -11,20 +11,19 @@
         <xacro:chassis/>
         <xacro:include filename="$(find rm_description)/urdf/common/imu.urdf.xacro"/>
-        <xacro:IMU connected_to="base_link" imu_name="base_imu" simulation="true"
-                   xyz="0.0 -0.165 0.0" rpy="0 0 0"/>
-    </xacro:if>
-    <xacro:if value="$(arg load_gimbal)">
-        <xacro:include filename="$(find rm_description)/urdf/standard/gimbal.urdf.xacro"/>
-        <xacro:include filename="$(find rm_description)/urdf/standard4/gimbal.transmission.urdf.xacro"/>
-        <xacro:include filename="$(find rm_description)/urdf/common/camera.urdf.xacro"/>
-        <xacro:camera_sensor xyz="0.127 0 -0.038" rpy="0 0 0" frame_id="$(arg camera_link)" parent="pitch"
-                             camera_sim="$(arg use_simulation)"/>
-        <xacro:camera_optical_frame xyz="0.088 -0.008 -0.043" rpy="1.583 -0.014 1.562"
-                                    frame_id="$(arg camera_optical_frame)" parent="pitch"
-                                    camera_sim="$(arg use_simulation)"/>
-    </xacro:if>
-    <xacro:if value="$(arg load_shooter)">
-        <xacro:include filename="$(find rm_description)/urdf/standard/shooter.urdf.xacro"/>
-        <xacro:include filename="$(find rm_description)/urdf/standard4/shooter.transmission.urdf.xacro"/>
+        <xacro:if value="$(arg load_gimbal)">
+            <xacro:include filename="$(find rm_description)/urdf/standard/gimbal.urdf.xacro"/>
+            <xacro:include filename="$(find rm_description)/urdf/standard4/gimbal.transmission.urdf.xacro"/>
+            <xacro:include filename="$(find rm_description)/urdf/common/camera.urdf.xacro"/>
+            <xacro:camera_sensor xyz="0.127 0 -0.038" rpy="0 0 0" frame_id="$(arg camera_link)" parent="pitch"
+                                 camera_sim="$(arg use_simulation)"/>
+            <xacro:camera_optical_frame xyz="0.088 -0.008 -0.043" rpy="1.583 -0.014 1.562"
+                                        frame_id="$(arg camera_optical_frame)" parent="pitch"
+                                        camera_sim="$(arg use_simulation)"/>
+            <xacro:IMU connected_to="pitch" imu_name="gimbal_imu" xyz="0.08 0. 0.08" rpy="0 0 -${pi/2}"/>
+            <xacro:if value="$(arg load_shooter)">
+                <xacro:include filename="$(find rm_description)/urdf/standard/shooter.urdf.xacro"/>
+                <xacro:include filename="$(find rm_description)/urdf/standard4/shooter.transmission.urdf.xacro"/>
+            </xacro:if>
+        </xacro:if>
     </xacro:if>
     <xacro:if value="$(arg use_simulation)">

File: rm_description/urdf/standard5/standard5.urdf.xacro (robot description, xacro)
@@ -11,21 +11,20 @@
         <xacro:include filename="$(find rm_description)/urdf/standard/chassis.urdf.xacro"/>
         <xacro:chassis roller_type="$(arg roller_type)"/>
-        <xacro:include filename="$(find rm_description)/urdf/common/imu.urdf.xacro"/>
-        <xacro:IMU connected_to="base_link" imu_name="base_imu" simulation="true"
-                   xyz="0.0 -0.165 0.0" rpy="0 0 0"/>
-    </xacro:if>
-    <xacro:if value="$(arg load_gimbal)">
-        <xacro:include filename="$(find rm_description)/urdf/standard/gimbal.urdf.xacro"/>
-        <xacro:include filename="$(find rm_description)/urdf/standard5/gimbal.transmission.urdf.xacro"/>
-        <xacro:include filename="$(find rm_description)/urdf/common/camera.urdf.xacro"/>
-        <xacro:camera_sensor xyz="0.127 0 -0.038" rpy="0 0 0" frame_id="$(arg camera_link)" parent="pitch"
-                             camera_sim="$(arg use_simulation)"/>
-        <xacro:camera_optical_frame xyz="0.089 -0.004 -0.083" rpy="1.593 0.0 1.567"
-                                    frame_id="$(arg camera_optical_frame)" parent="pitch"
-                                    camera_sim="$(arg use_simulation)"/>
-    </xacro:if>
-    <xacro:if value="$(arg load_shooter)">
-        <xacro:include filename="$(find rm_description)/urdf/standard/shooter.urdf.xacro"/>
-        <xacro:include filename="$(find rm_description)/urdf/standard5/shooter.transmission.urdf.xacro"/>
+        <xacro:if value="$(arg load_gimbal)">
+            <xacro:include filename="$(find rm_description)/urdf/standard/gimbal.urdf.xacro"/>
+            <xacro:include filename="$(find rm_description)/urdf/standard5/gimbal.transmission.urdf.xacro"/>
+            <!--            <xacro:include filename="$(find rm_description)/urdf/common/camera.urdf.xacro"/>-->
+            <!--            <xacro:camera_sensor xyz="0.127 0 -0.038" rpy="0 0 0" frame_id="$(arg camera_link)" parent="pitch"-->
+            <!--                                 camera_sim="$(arg use_simulation)"/>-->
+            <!--            <xacro:camera_optical_frame xyz="0.089 -0.004 -0.083" rpy="1.593 0.0 1.567"-->
+            <!--                                        frame_id="$(arg camera_optical_frame)" parent="pitch"-->
+            <!--                                        camera_sim="$(arg use_simulation)"/>-->
+            <xacro:include filename="$(find rm_description)/urdf/common/imu.urdf.xacro"/>
+            <xacro:IMU connected_to="pitch" imu_name="gimbal_imu" xyz="0.08 0. 0.08" rpy="0 0 -${pi/2}"/>
+            <xacro:if value="$(arg load_shooter)">
+                <xacro:include filename="$(find rm_description)/urdf/standard/shooter.urdf.xacro"/>
+                <xacro:include filename="$(find rm_description)/urdf/standard5/shooter.transmission.urdf.xacro"/>
+            </xacro:if>
+        </xacro:if>
     </xacro:if>
     <xacro:if value="$(arg use_simulation)">
