Commit message: Rebase from 'upstream'

File: rm_description/urdf/balance/balance.urdf.xacro (robot description, xacro)
@@ -8,4 +8,5 @@
         <xacro:include filename="$(find rm_description)/urdf/balance/chassis.urdf.xacro"/>
         <xacro:chassis/>
+        <xacro:include filename="$(find rm_description)/urdf/common/imu.urdf.xacro"/>
         <xacro:IMU connected_to="base_link" imu_name="base_imu" xyz="0.08 0. 0.08" rpy="0 0 0"/>
         <xacro:if value="$(arg load_gimbal)">

File: rm_description/urdf/common/imu.urdf.xacro (robot description, xacro)
@@ -11,7 +11,7 @@
         <link name="${imu_name}">
             <inertial>
-                <mass value="0.001"/>
+                <mass value="0.01"/>
                 <origin rpy="0 0 0" xyz="0 0 0"/>
-                <inertia ixx="0.0001" ixy="0" ixz="0" iyy="0.000001" iyz="0" izz="0.0001"/>
+                <inertia ixx="0.000001" ixy="0" ixz="0" iyy="0.000001" iyz="0" izz="0.000001"/>
             </inertial>
             <visual>

File: rm_description/urdf/common/swerve_drive.urdf.xacro (robot description, xacro)
@@ -18,14 +18,14 @@
             <inertial>
                 <xacro:if value="${reflect == 1}">
-                    <mass value="3.725118"/>
-                    <origin xyz="0.951e-3 5.254e-3 -23.161e-3" rpy="0 0 0"/>
-                    <inertia ixx="1.645e-2" ixy="-13783.466e-9" ixz="2.345e-4" iyy="1.562e-2" iyz="2.132e-3"
-                             izz="3.256e-3"/>
+                    <mass value="0.854"/>
+                    <origin xyz="0.000054 0.008 0.00548" rpy="0 0 0"/>
+                    <inertia ixx="6.711e-4" ixy="1.958e-9" ixz="-1.109e-6" iyy="6.703e-4" iyz="-1.095e-7"
+                             izz="7.091e-4"/>
                 </xacro:if>
                 <xacro:if value="${reflect == -1}">
-                    <mass value="3.725115"/>
-                    <origin xyz="0.156793 0.150588 0.030271" rpy="0 0 0"/>
-                    <inertia ixx="1.143e-1" ixy="-9.835e-2" ixz="-2.178e-2" iyy="1.207e-1" iyz="-2.289e-2"
-                             izz="2e-1"/>
+                    <mass value="0.854"/>
+                    <origin xyz="0.000054 0.008 0.00548" rpy="0 0 0"/>
+                    <inertia ixx="6.711e-4" ixy="1.958e-9" ixz="-1.109e-6" iyy="6.703e-4" iyz="-1.095e-7"
+                             izz="7.091e-4"/>
                 </xacro:if>
             </inertial>
@@ -66,7 +66,7 @@
             </visual>
             <inertial>
-                <mass value="0.18791"/>
-                <origin xyz="6.908e-8 -7.298e-3 275e-6" rpy="0 0 0"/>
-                <inertia ixx="1.584e-4" ixy="0.199e-9" ixz="-0.173e-9" iyy="2.141e-4" iyz="768.622e-9" izz="1.575e-4"/>
+                <mass value="0.543"/>
+                <origin xyz="0.000024 0.024 0.000129" rpy="0 0 0"/>
+                <inertia ixx="4.895e-4" ixy="-3.948e-7" ixz="1.726e-7" iyy="2.894e-4" iyz="1.133e-6" izz="4.887e-4"/>
             </inertial>
             <collision>

File: rm_description/urdf/rmua/gimbal.transmission.urdf.xacro (robot description, xacro)
@@ -7,5 +7,5 @@
         </actuator>
         <joint name="yaw_joint">
-            <offset>0.417</offset>
+            <offset>-3.675</offset>
             <hardwareInterface>hardware_interface/EffortJointInterface</hardwareInterface>
         </joint>
@@ -17,5 +17,5 @@
         </actuator>
         <joint name="pitch_joint">
-            <offset>1.559</offset>
+            <offset>4.779</offset>
             <hardwareInterface>hardware_interface/EffortJointInterface</hardwareInterface>
         </joint>

File: rm_description/urdf/rmua/gimbal.urdf.xacro (robot description, xacro)
@@ -2,6 +2,8 @@
 <robot xmlns:xacro="http://www.ros.org/wiki/xacro">
     <xacro:property name="threshold" value="0.1"/>
-    <xacro:property name="pitch_lower_limit" value="-0.7"/>
-    <xacro:property name="pitch_upper_limit" value="0.4"/>
+    <xacro:property name="pitch_lower_limit" value="-0.482"/>
+    <xacro:property name="pitch_upper_limit" value="0.394"/>
+    <xacro:property name="yaw_lower_limit" value="-1.732"/>
+    <xacro:property name="yaw_upper_limit" value="1.674"/>
     <link name="yaw">
         <inertial>
@@ -28,5 +30,8 @@
                 rpy="0 0 0"/>
         <dynamics damping="0.0" friction="0.1"/>
-        <limit effort="1.2" velocity="31" lower="-1e10" upper="1e10"/>
+        <limit effort="1.2" velocity="31" lower="${yaw_lower_limit}" upper="${yaw_upper_limit}"/>
+        <safety_controller k_position="100" k_velocity="0.1"
+                           soft_lower_limit="${yaw_lower_limit+threshold}"
+                           soft_upper_limit="${yaw_upper_limit-threshold}"/>
         <parent link="base_link"/>
         <child link="yaw"/>

File: rm_description/urdf/rmua/shooter.urdf.xacro (robot description, xacro)
@@ -33,5 +33,5 @@
     </link>
     <joint name="trigger_joint" type="continuous">
-        <origin xyz="-0.068.666 -0.0145 0.0624" rpy="0 0 0"/>
+        <origin xyz="-0.068 -0.0145 0.0624" rpy="0 0 0"/>
         <dynamics damping="0.0" friction="0.01"/>
         <limit effort="1.0" velocity="43.54" lower="-1e16" upper="1e16"/>

File: rm_description/urdf/standard/chassis.urdf.xacro (robot description, xacro)
@@ -8,8 +8,8 @@
         <link name="base_link">
             <inertial>
-                <mass value="10.56"/>
-                <origin xyz="-0.025077  0  0.055047"/>
-                <inertia ixx="2.247e-1" ixy="-1.139e-5" ixz="2.983e-2" iyy="3.771e-1"
-                         iyz="3.3454e-6" izz="4.803e-1"/>
+                <mass value="1.737"/>
+                <origin xyz="0.000425  -0.000733  0.00762"/>
+                <inertia ixx="4.088e-2" ixy="9.103e-5" ixz="-1.697e-4" iyy="4.498e-2"
+                         iyz="6.472e-5" izz="8.107e-2"/>
             </inertial>
             <visual>

File: rm_description/urdf/standard/gimbal.urdf.xacro (robot description, xacro)
@@ -6,8 +6,8 @@
         <link name="yaw">
             <inertial>
-                <mass value="0.592087"/>
-                <origin xyz="0 0 0.0127"/>
-                <inertia ixx="6.17e-4" ixy="0." ixz="0." iyy="6.182e-4"
-                         iyz="0." izz="1.07e-3"/>
+                <mass value="1.337"/>
+                <origin xyz="0.00072 0.000098 0.00976"/>
+                <inertia ixx="4.777e-3" ixy="-1.108e-5" ixz="1.574e-5" iyy="4.902e-3"
+                         iyz="-1.234e-5" izz="3.643e-3"/>
             </inertial>
             <visual>
@@ -35,8 +35,8 @@
         <link name="pitch">
             <inertial>
-                <mass value="1.475"/>
-                <origin xyz="0.0168 -0.0028 0.0225"/>
-                <inertia ixx="5.619e-3" ixy="1.192e-4" ixz="-1.795e-4" iyy="6.577e-3"
-                         iyz="8.931e-5" izz="6.867e-3"/>
+                <mass value="1.175"/>
+                <origin xyz="-0.00439 0.0113 -0.00970"/>
+                <inertia ixx="4.716e-3" ixy="-1.511e-4" ixz="-1.134e-4" iyy="5.220e-3"
+                         iyz="1.192e-5" izz="6.046e-3"/>
             </inertial>
             <visual>

File: rm_description/urdf/standard/shooter.urdf.xacro (robot description, xacro)
@@ -13,8 +13,8 @@
     <link name="trigger">
         <inertial>
-            <mass value="0.295177"/>
-            <origin xyz="-0.00842 0.0 0.00605"/>
-            <inertia ixx="2.255e-4" ixy="2.5698e-7" ixz="2.3929e-6" iyy="2.233e-4"
-                     iyz="5.22e-7" izz="2.643e-4"/>
+            <mass value="0.2972"/>
+            <origin xyz="-0.00549 -0.00233 0.00344"/>
+            <inertia ixx="1.955e-4" ixy="-2.402e-5" ixz="-2.718e-5" iyy="3.514e-4"
+                     iyz="-6.239e-6" izz="4.209e-4"/>
         </inertial>
         <visual>

File: rm_description/urdf/standard3/standard3.urdf.xacro (robot description, xacro)
@@ -11,5 +11,4 @@
         <xacro:include filename="$(find rm_description)/urdf/standard/chassis.urdf.xacro"/>
         <xacro:chassis roller_type="$(arg roller_type)"/>
-        <xacro:include filename="$(find rm_description)/urdf/common/imu.urdf.xacro"/>
         <xacro:if value="$(arg load_gimbal)">
             <xacro:include filename="$(find rm_description)/urdf/standard/gimbal.urdf.xacro"/>

File: rm_description/urdf/standard4/chassis.urdf.xacro (robot description, xacro)
@@ -8,8 +8,8 @@
         <link name="base_link">
             <inertial>
-                <mass value="35.539863"/>
-                <origin xyz="-0.032179 0.015648 0.0968"/>
-                <inertia ixx="1.519" ixy="4.205e-2" ixz="2.407e-1" iyy="1.668"
-                         iyz="8.007e-2" izz="1.891"/>
+                <mass value="1.737"/>
+                <origin xyz="0.000425  -0.000733  0.00762"/>
+                <inertia ixx="4.088e-2" ixy="9.103e-5" ixz="-1.697e-4" iyy="4.498e-2"
+                         iyz="6.472e-5" izz="8.107e-2"/>
             </inertial>
             <visual>

File: rm_description/urdf/standard4/standard4.urdf.xacro (robot description, xacro)
@@ -10,15 +10,15 @@
         <xacro:include filename="$(find rm_description)/urdf/standard4/chassis.urdf.xacro"/>
         <xacro:chassis/>
-        <xacro:include filename="$(find rm_description)/urdf/common/imu.urdf.xacro"/>
         <xacro:if value="$(arg load_gimbal)">
             <xacro:include filename="$(find rm_description)/urdf/standard/gimbal.urdf.xacro"/>
             <xacro:include filename="$(find rm_description)/urdf/standard4/gimbal.transmission.urdf.xacro"/>
-            <xacro:include filename="$(find rm_description)/urdf/common/camera.urdf.xacro"/>
-            <xacro:camera_sensor xyz="0.127 0 -0.038" rpy="0 0 0" frame_id="$(arg camera_link)" parent="pitch"
-                                 camera_sim="$(arg use_simulation)"/>
-            <xacro:camera_optical_frame xyz="0.088 -0.008 -0.043" rpy="1.583 -0.014 1.562"
-                                        frame_id="$(arg camera_optical_frame)" parent="pitch"
-                                        camera_sim="$(arg use_simulation)"/>
-            <xacro:IMU connected_to="pitch" imu_name="gimbal_imu" xyz="0.08 0. 0.08" rpy="0 0 -${pi/2}"/>
+            <!--            <xacro:include filename="$(find rm_description)/urdf/common/camera.urdf.xacro"/>-->
+            <!--            <xacro:camera_sensor xyz="0.127 0 -0.038" rpy="0 0 0" frame_id="$(arg camera_link)" parent="pitch"-->
+            <!--                                 camera_sim="$(arg use_simulation)"/>-->
+            <!--            <xacro:camera_optical_frame xyz="0.089 -0.004 -0.083" rpy="1.593 0.0 1.567"-->
+            <!--                                        frame_id="$(arg camera_optical_frame)" parent="pitch"-->
+            <!--                                        camera_sim="$(arg use_simulation)"/>-->
+            <xacro:include filename="$(find rm_description)/urdf/common/imu.urdf.xacro"/>
+            <xacro:IMU connected_to="pitch" imu_name="gimbal_imu" xyz="0.08 0. 0.08" rpy="0 0 0"/>
             <xacro:if value="$(arg load_shooter)">
                 <xacro:include filename="$(find rm_description)/urdf/standard/shooter.urdf.xacro"/>

File: rm_description/urdf/standard5/standard5.urdf.xacro (robot description, xacro)
@@ -21,5 +21,5 @@
             <!--                                        camera_sim="$(arg use_simulation)"/>-->
             <xacro:include filename="$(find rm_description)/urdf/common/imu.urdf.xacro"/>
-            <xacro:IMU connected_to="pitch" imu_name="gimbal_imu" xyz="0.08 0. 0.08" rpy="0 0 -${pi/2}"/>
+            <xacro:IMU connected_to="pitch" imu_name="gimbal_imu" xyz="0.08 0. 0.08" rpy="${pi} 0 0"/>
             <xacro:if value="$(arg load_shooter)">
                 <xacro:include filename="$(find rm_description)/urdf/standard/shooter.urdf.xacro"/>
